File: Debug Adapter/Debug Adapter.kicad_sch (KiCad schematic)
At the start: 8 parts, among them J1 Conn_01x03_Pin, J2 Conn_01x06_Pin, J3 Conn_01x06_Socket, U1 VOD207T

Commit message: More temperature adjustments
Connections:
- net RXD: now also R3.1, U1.6; no longer U1.3
- net TXD: now also U1.2; no longer R4.1, U1.8
- net at R2.2: now also U1.3; no longer U1.4
- removed net RXD MCU: J1.2 (Pin_2), R3.1, U1.6
- net TXD MCU renamed TXD Reflow
- net TXD Reflow: now also U1.4; no longer U1.2
- new net RXD Reflow: J1.2 (Pin_2), R4.1, U1.8
Other:
- moved on the sheet: R2
Changed lines of the file:
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@@
-	(wire
-		(pts
-			(xy 104.14 87.63) (xy 106.68 87.63)
-		)
-		(stroke
-			(width 0)
-			(type default)
-		)
-	)
 	(wire
 		(pts
@@
 	(wire
 		(pts
+			(xy 104.14 82.55) (xy 106.68 82.55)
+		)
+		(stroke
+			(width 0)
+			(type default)
+		)
+	)
+	(wire
+		(pts
 			(xy 147.32 74.93) (xy 144.78 74.93)
 		)
@@
 		)
 	)
-	(global_label "TXD MCU"
+	(text_box "Transmit and Receive are swapped internally to match the connections to the PCB Reflow Plate"
+		(exclude_from_sim no)
+		(at 104.14 93.98 0)
+		(size 53.34 7.62)
+		(stroke
+			(width 0)
+			(type default)
+		)
+		(fill
+			(type color)
+			(color 255 255 194 1)
+		)
+		(effects
+			(font
+				(size 1.27 1.27)
+			)
+			(justify left top)
+		)
+	)
+	(global_label "TXD"
 		(shape input)
 		(at 114.3 77.47 180)
@@
 		)
 		(property "Intersheetrefs" "${INTERSHEET_REFS}"
-			(at 102.8482 77.47 0)
+			(at 107.8677 77.47 0)
 			(effects
 				(font
@@
 		)
 	)
-	(global_label "RXD MCU"
+	(global_label "RXD"
 		(shape input)
 		(at 147.32 85.09 0)
@@
 		)
 		(property "Intersheetrefs" "${INTERSHEET_REFS}"
-			(at 159.0742 85.09 0)
+			(at 154.0547 85.09 0)
 			(effects
 				(font
@@
 		)
 	)
-	(global_label "TXD MCU"
+	(global_label "TXD Reflow"
 		(shape input)
 		(at 107.95 111.76 270)
@@
 		)
 		(property "Intersheetrefs" "${INTERSHEET_REFS}"
-			(at 107.95 123.2118 90)
+			(at 107.95 125.3889 90)
 			(effects
 				(font
@@
 		)
 	)
+	(global_label "TXD Reflow"
+		(shape input)
+		(at 114.3 87.63 180)
+		(fields_autoplaced yes)
+		(effects
+			(font
+				(size 1.27 1.27)
+			)
+			(justify right)
+		)
+		(property "Intersheetrefs" "${INTERSHEET_REFS}"
+			(at 100.6711 87.63 0)
+			(effects
+				(font
+					(size 1.27 1.27)
+				)
+				(justify right)
+				(hide yes)
+			)
+		)
+	)
+	(global_label "RTS"
+		(shape input)
+		(at 121.92 111.76 270)
+		(fields_autoplaced yes)
+		(effects
+			(font
+				(size 1.27 1.27)
+			)
+			(justify right)
+		)
+		(property "Intersheetrefs" "${INTERSHEET_REFS}"
+			(at 121.92 118.1923 90)
+			(effects
+				(font
+					(size 1.27 1.27)
+				)
+				(justify right)
+				(hide yes)
+			)
+		)
+	)
+	(global_label "RXD Reflow"
+		(shape input)
+		(at 110.49 111.76 270)
+		(fields_autoplaced yes)
+		(effects
+			(font
+				(size 1.27 1.27)
+			)
+			(justify right)
+		)
+		(property "Intersheetrefs" "${INTERSHEET_REFS}"
+			(at 110.49 125.6913 90)
+			(effects
+				(font
+					(size 1.27 1.27)
+				)
+				(justify right)
+				(hide yes)
+			)
+		)
+	)
 	(global_label "RXD"
 		(shape input)
-		(at 114.3 82.55 180)
-		(fields_autoplaced yes)
-		(effects
-			(font
-				(size 1.27 1.27)
-			)
-			(justify right)
-		)
-		(property "Intersheetrefs" "${INTERSHEET_REFS}"
-			(at 107.5653 82.55 0)
-			(effects
-				(font
-					(size 1.27 1.27)
-				)
-				(justify right)
-				(hide yes)
-			)
-		)
-	)
-	(global_label "RTS"
-		(shape input)
-		(at 121.92 111.76 270)
-		(fields_autoplaced yes)
-		(effects
-			(font
-				(size 1.27 1.27)
-			)
-			(justify right)
-		)
-		(property "Intersheetrefs" "${INTERSHEET_REFS}"
-			(at 121.92 118.1923 90)
-			(effects
-				(font
-					(size 1.27 1.27)
-				)
-				(justify right)
-				(hide yes)
-			)
-		)
-	)
-	(global_label "RXD MCU"
-		(shape input)
-		(at 110.49 111.76 270)
-		(fields_autoplaced yes)
-		(effects
-			(font
-				(size 1.27 1.27)
-			)
-			(justify right)
-		)
-		(property "Intersheetrefs" "${INTERSHEET_REFS}"
-			(at 110.49 123.5142 90)
-			(effects
-				(font
-					(size 1.27 1.27)
-				)
-				(justify right)
-				(hide yes)
-			)
-		)
-	)
-	(global_label "RXD"
-		(shape input)
 		(at 148.59 111.76 270)
 		(fields_autoplaced yes)
@@
 		)
 	)
-	(global_label "TXD"
+	(global_label "RXD Reflow"
 		(shape input)
 		(at 147.32 74.93 0)
@@
 		)
 		(property "Intersheetrefs" "${INTERSHEET_REFS}"
-			(at 153.7523 74.93 0)
+			(at 161.2513 74.93 0)
 			(effects
 				(font
@@
 	(symbol
 		(lib_id "Device:R")
-		(at 110.49 87.63 90)
+		(at 110.49 82.55 90)
 		(unit 1)
 		(exclude_from_sim no)
@@
 		(dnp no)
 		(property "Reference" "R2"
-			(at 110.49 89.662 90)
+			(at 110.49 80.518 90)
 			(effects
 				(font
@@
 		)
 		(property "Value" "470R"
-			(at 110.49 92.202 90)
+			(at 110.744 84.836 90)
 			(effects
 				(font
@@
 		)
 		(property "Footprint" "Resistor_SMD:R_0402_1005Metric"
-			(at 110.49 89.408 90)
+			(at 110.49 84.328 90)
 			(effects
 				(font
@@
 		)
 		(property "Datasheet" "~"
-			(at 110.49 87.63 0)
+			(at 110.49 82.55 0)
 			(effects
 				(font
@@
 		)
 		(property "Description" "Resistor"
-			(at 110.49 87.63 0)
+			(at 110.49 82.55 0)
 			(effects
 				(font
@@
 	(symbol
 		(lib_id "power:+5V")
-		(at 104.14 87.63 0)
+		(at 104.14 82.55 0)
 		(unit 1)
 		(exclude_from_sim no)
@@
 		(fields_autoplaced yes)
 		(property "Reference" "#PWR02"
-			(at 104.14 91.44 0)
+			(at 104.14 86.36 0)
 			(effects
 				(font
@@
 		)
 		(property "Value" "+5V"
+			(at 104.14 77.47 0)
+			(effects
+				(font
+					(size 1.27 1.27)
+				)
+			)
+		)
+		(property "Footprint" ""
 			(at 104.14 82.55 0)
 			(effects
@@
 					(size 1.27 1.27)
 				)
-			)
-		)
-		(property "Footprint" ""
-			(at 104.14 87.63 0)
-			(effects
-				(font
-					(size 1.27 1.27)
-				)
 				(hide yes)
 			)
 		)
 		(property "Datasheet" ""
-			(at 104.14 87.63 0)
+			(at 104.14 82.55 0)
 			(effects
 				(font
@@
 		)
 		(property "Description" "Power symbol creates a global label with name \"+5V\""
-			(at 104.14 87.63 0)
-			(effects
-				(font
+			(at 104.14 82.55 0)
+			(effects
+				(font
